Commit message: error in desc

File: mse6_description/urdf/mse6_description.urdf (robot description, URDF)
Before this commit: robot mse6_description, 10 links, 8 joints
Joints:
- added joint fwd_left_wheel_holder_j: type revolute, parent body_upper_link, child fwd_left_wheel_holder_link, origin xyz=-0.1 -0.054 0.065 rpy=0 0 0.035451, axis 0 0 1, limit lower=-0.5 upper=0.5 effort=0.5 velocity=0.5

Commit message: fix export

File: mse6_description/urdf/mse6_description.urdf (robot description, URDF)
Before this commit: robot mse6_description, 10 links, 9 joints
Links:
- link body_bott_link: mass 0.669776829617328 -> 0.669776829617329

Commit message: fixed links and joints

File: mse6_description/urdf/mse6_description.urdf (robot description, URDF)
Before this commit: robot mse6_description, 10 links, 9 joints
Joints:
- joint back_left_wheel_j: axis 0 0 0 -> 0 1 0
- joint back_right_wheel_j: axis 0 0 0 -> 0 1 0
- joint fwd_left_wheel_holder_j: axis 0 0 1 -> 0 1 0
- joint fwd_left_wheel_j: axis 0 0 0 -> 0 1 0
- joint fwd_right_wheel_holder_j: axis 0 0 0 -> 0 1 0
- joint fwd_right_wheel_j: axis 0 0 0 -> 0 1 0

Commit message: true base link added

File: mse6_description/urdf/mse6_description.urdf (robot description, URDF)
Before this commit: robot mse6_description, 10 links, 9 joints
Links:
- added link base_link
Joints:
- added joint body_bott_link_j: type fixed, parent base_link, child body_bott_link, origin xyz=0 0 0.055 rpy=0 0 3.1416

Commit message: added fake links for steer

File: mse6_description/urdf/mse6_description.urdf (robot description, URDF)
Before this commit: robot mse6_description, 11 links, 10 joints
Links:
- added link fake_back_wheel_link
- added link fake_fwd_wheel_link
Joints:
- added joint fake_back_wheel_j: type fixed, parent body_upper_link, child fake_back_wheel_link, origin xyz=0.1 -0.054 0.0 rpy=1.5707 0 3.1415
- added joint fake_fwd_wheel_j: type fixed, parent body_upper_link, child fake_fwd_wheel_link, origin xyz=-0.1 -0.054 0 rpy=1.5707 0 3.1415

Commit message: controller spawner could not find interface

File: mse6_description/urdf/mse6_description.urdf (robot description, URDF)
Before this commit: robot mse6_description, 13 links, 12 joints
Joints:
- joint fake_back_wheel_j: axis (none) -> 0 1 0; type fixed -> continuous
- joint fake_fwd_wheel_j: axis (none) -> 0 0 1; limit (none) -> lower=-0.5 upper=0.5 effort=0.5 velocity=0.5; type fixed -> revolute
