Commit message: not it is riding but wierd

File: mse6_description/urdf/mse6.xacro (robot description, xacro)
@@ -3,7 +3,8 @@
      Commit Version: 1.6.0-1-g15f4949  Build Version: 1.6.7594.29634
      For more information, please see http://wiki.ros.org/sw_urdf_exporter -->
-<robot
-  name="mse6" xmlns:xacro="http://www.ros.org/wiki/xacro">
+<robot xmlns:xacro="http://www.ros.org/wiki/xacro" name="mse6">
   <xacro:include filename="$(find mse6_description)/urdf/mse6.gazebo"/>
+  <xacro:property name="wheel_r" value="0.025"/>
+  <xacro:property name="wheel_h" value="0.030"/>
   <link name="base_link"/>
   <joint name="body_bott_link_j"
@@ -218,9 +219,10 @@
     <collision>
       <origin
-        xyz="0 0 0"
-        rpy="0 0 0" />
-      <geometry>
-        <mesh
-          filename="package://mse6_description/meshes/fwd_left_wheel_link.STL" />
+        xyz="0 ${wheel_h/2} 0"
+        rpy="${pi/2} 0 0" />
+      <geometry>
+        <!--<mesh
+          filename="package://mse6_description/meshes/fwd_left_wheel_link.STL" />-->
+          <cylinder length="${wheel_h}" radius="${wheel_r}"/>
       </geometry>
     </collision>
@@ -252,5 +254,5 @@
     </actuator>
   </transmission>
-  <transmission name="tran_fwd_left">
+  <!--<transmission name="tran_fwd_left">
     <type>transmission_interface/SimpleTransmission</type>
     <joint name="fwd_left_wheel_j">
@@ -261,5 +263,5 @@
         <mechanicalReduction>1</mechanicalReduction>
     </actuator>
-  </transmission>
+  </transmission>-->
   <!-- FORWARD RIGHT WHEEL -->
   <link
@@ -356,9 +358,10 @@
     <collision>
       <origin
-        xyz="0 0 0"
-        rpy="0 0 0" />
-      <geometry>
-        <mesh
-          filename="package://mse6_description/meshes/fwd_right_wheel_link.STL" />
+        xyz="0 ${wheel_h/2} 0"
+        rpy="${pi/2} 0 0" />
+      <geometry>
+        <!--<mesh
+          filename="package://mse6_description/meshes/fwd_left_wheel_link.STL" />-->
+          <cylinder length="${wheel_h}" radius="${wheel_r}"/>
       </geometry>
     </collision>
@@ -390,5 +393,5 @@
     </actuator>
   </transmission>
-  <transmission name="tran_fwd_right">
+  <!--<transmission name="tran_fwd_right">
     <type>transmission_interface/SimpleTransmission</type>
     <joint name="fwd_right_wheel_j">
@@ -399,5 +402,5 @@
         <mechanicalReduction>1</mechanicalReduction>
     </actuator>
-  </transmission>
+  </transmission>-->
   <!-- FAKE BACK LINK -->
   <link name="fake_back_wheel_link"/>
@@ -496,9 +499,10 @@
     <collision>
       <origin
-        xyz="0 0 0"
-        rpy="0 0 0" />
-      <geometry>
-        <mesh
-          filename="package://mse6_description/meshes/back_left_wheel_link.STL" />
+        xyz="0 ${wheel_h/2} 0"
+        rpy="${pi/2} 0 0" />
+      <geometry>
+        <!--<mesh
+          filename="package://mse6_description/meshes/fwd_left_wheel_link.STL" />-->
+          <cylinder length="${wheel_h}" radius="${wheel_r}"/>
       </geometry>
     </collision>
@@ -626,9 +630,10 @@
     <collision>
       <origin
-        xyz="0 0 0"
-        rpy="0 0 0" />
-      <geometry>
-        <mesh
-          filename="package://mse6_description/meshes/back_right_wheel_link.STL" />
+        xyz="0 ${wheel_h/2} 0"
+        rpy="${pi/2} 0 0" />
+      <geometry>
+        <!--<mesh
+          filename="package://mse6_description/meshes/fwd_left_wheel_link.STL" />-->
+          <cylinder length="${wheel_h}" radius="${wheel_r}"/>
       </geometry>
     </collision>
@@ -645,5 +650,5 @@
       link="back_right_wheel_link" />
     <axis
-      xyz="0 1 0" />
+      xyz="0 -1 0" />
     <dynamics
       damping="0.01"
@@ -670,3 +675,9 @@
         </actuator>
     </transmission>
+    <!--<gazebo>
+    <plugin name="gazebo_ros_control" filename="libgazebo_ros_control.so">
+      <robotNamespace></robotNamespace>
+      <robotSimType>steer_bot_hardware_gazebo/SteerBotHardwareGazebo</robotSimType>
+    </plugin>
+  </gazebo>-->
 </robot>

Commit message: to left turn is ok, but not good for turn right

File: mse6_description/urdf/mse6.xacro (robot description, xacro)
@@ -50,8 +50,8 @@
         xyz="0 0 0"
         rpy="0 0 0" />
-      <geometry>
+      <!--<geometry>
         <mesh
           filename="package://mse6_description/meshes/body_bott_link.STL" />
-      </geometry>
+      </geometry>-->
     </collision>
   </link>
@@ -118,5 +118,5 @@
           rpy="1.5707 0 3.1415"
           />
-      <axis xyz="0 0 1"/>
+      <axis xyz="0 1 0"/>
       <limit
         lower="-0.5"

Commit message: reorginized

File: mse6_description/urdf/mse6.xacro (robot description, xacro)
@@ -50,8 +50,8 @@
         xyz="0 0 0"
         rpy="0 0 0" />
-      <!--<geometry>
+      <geometry>
         <mesh
           filename="package://mse6_description/meshes/body_bott_link.STL" />
-      </geometry>-->
+      </geometry>
     </collision>
   </link>

Commit message: nav works somehow

File: mse6_description/urdf/mse6.xacro (robot description, xacro)
@@ -7,4 +7,5 @@
   <xacro:property name="wheel_r" value="0.025"/>
   <xacro:property name="wheel_h" value="0.030"/>
+  <xacro:property name="steer_limit" value="0.5"/>
   <link name="base_link"/>
   <joint name="body_bott_link_j"
@@ -120,6 +121,6 @@
       <axis xyz="0 1 0"/>
       <limit
-        lower="-0.5"
-        upper="0.5"
+        lower="${-steer_limit}"
+        upper="${steer_limit}"
         effort="0.5"
         velocity="0.5" />
@@ -179,6 +180,6 @@
       xyz="0 1 0" />
     <limit
-      lower="-0.5"
-      upper="0.5"
+      lower="${-steer_limit}"
+      upper="${steer_limit}"
       effort="0.5"
       velocity="0.5" />

Commit message: added laser scanner

File: mse6_description/urdf/mse6.xacro (robot description, xacro)
@@ -9,4 +9,14 @@
   <xacro:property name="steer_limit" value="0.5"/>
   <link name="base_link"/>
+  <link name="laser_scanner_link"/>
+  <joint name="laser_scanner_j"
+         type="fixed">
+      <parent link="base_link"/>
+      <child link="laser_scanner_link"/>
+      <origin
+          xyz="0.1 0 0.07"
+          rpy="0 0 0"/>
+  </joint>
+  <!-- BODY -->
   <joint name="body_bott_link_j"
          type="fixed">

Commit message: holocamera added to nav stack

File: mse6_description/urdf/mse6.xacro (robot description, xacro)
@@ -9,4 +9,5 @@
   <xacro:property name="steer_limit" value="0.5"/>
   <link name="base_link"/>
+  <!-- SENSORS -->
   <link name="laser_scanner_link"/>
   <joint name="laser_scanner_j"
@@ -18,4 +19,22 @@
           rpy="0 0 0"/>
   </joint>
+  <link name="holocamera_link"/>
+  <joint name="holocamera_j"
+         type="fixed">
+      <parent link="base_link"/>
+      <child link="holocamera_link"/>
+      <origin
+          xyz="0.19 0 0.07"
+          rpy="0 0 0"/>
+  </joint>
+  <link name="holocamera_optical_link"/>
+  <joint name="holocamera_optical_j"
+         type="fixed">
+      <parent link="holocamera_link"/>
+      <child link="holocamera_optical_link"/>
+      <origin
+          xyz="0 0 0"
+          rpy="${-pi/2} 0 ${-pi/2}"/>
+  </joint>
   <!-- BODY -->
   <joint name="body_bott_link_j"
@@ -25,5 +44,5 @@
       <origin
           xyz = "0 0 0.055"
-          rpy="0 0 3.1416"/>
+          rpy="0 0 ${pi}"/>
   </joint>
   <link
@@ -127,5 +146,5 @@
       <origin
           xyz="-0.1 -0.054 0"
-          rpy="1.5707 0 3.1415"
+          rpy="${pi/2} 0 ${pi}"
           />
       <axis xyz="0 1 0"/>
@@ -419,5 +438,5 @@
          <origin
              xyz="0.1 -0.054 0.0"
-             rpy="1.5707 0 3.1415"/>
+             rpy="${pi/2} 0 ${pi}"/>
          <parent link="body_upper_link"/>
          <child link="fake_back_wheel_link"/>

Commit message: mse bot now every thing seems in namespace

File: mse6_description/urdf/mse6.xacro (robot description, xacro)
@@ -4,33 +4,34 @@
      For more information, please see http://wiki.ros.org/sw_urdf_exporter -->
 <robot xmlns:xacro="http://www.ros.org/wiki/xacro" name="mse6">
+  <xacro:arg name="robot" default="mse6-XXXXX"/>
   <xacro:include filename="$(find mse6_description)/urdf/mse6.gazebo"/>
   <xacro:property name="wheel_r" value="0.025"/>
   <xacro:property name="wheel_h" value="0.030"/>
   <xacro:property name="steer_limit" value="0.5"/>
-  <link name="base_link"/>
+  <link name="$(arg robot)/base_link"/>
   <!-- SENSORS -->
-  <link name="laser_scanner_link"/>
-  <joint name="laser_scanner_j"
+  <link name="$(arg robot)/laser_scanner_link"/>
+  <joint name="$(arg robot)/laser_scanner_j"
          type="fixed">
-      <parent link="base_link"/>
-      <child link="laser_scanner_link"/>
+      <parent link="$(arg robot)/base_link"/>
+      <child link="$(arg robot)/laser_scanner_link"/>
       <origin
           xyz="0.1 0 0.07"
           rpy="0 0 0"/>
   </joint>
-  <link name="holocamera_link"/>
-  <joint name="holocamera_j"
+  <link name="$(arg robot)/holocamera_link"/>
+  <joint name="$(arg robot)/holocamera_j"
          type="fixed">
-      <parent link="base_link"/>
-      <child link="holocamera_link"/>
+      <parent link="$(arg robot)/base_link"/>
+      <child link="$(arg robot)/holocamera_link"/>
       <origin
           xyz="0.19 0 0.07"
           rpy="0 0 0"/>
   </joint>
-  <link name="holocamera_optical_link"/>
-  <joint name="holocamera_optical_j"
+  <link name="$(arg robot)/holocamera_optical_link"/>
+  <joint name="$(arg robot)/holocamera_optical_j"
          type="fixed">
-      <parent link="holocamera_link"/>
-      <child link="holocamera_optical_link"/>
+      <parent link="$(arg robot)/holocamera_link"/>
+      <child link="$(arg robot)/holocamera_optical_link"/>
       <origin
           xyz="0 0 0"
@@ -38,8 +39,8 @@
   </joint>
   <!-- BODY -->
-  <joint name="body_bott_link_j"
+  <joint name="$(arg robot)/body_bott_link_j"
          type="fixed">
-      <parent link="base_link"/>
-      <child link="body_bott_link"/>
+      <parent link="$(arg robot)/base_link"/>
+      <child link="$(arg robot)/body_bott_link"/>
       <origin
           xyz = "0 0 0.055"
@@ -47,5 +48,5 @@
   </joint>
   <link
-    name="body_bott_link">
+    name="$(arg robot)/body_bott_link">
     <inertial>
       <origin
@@ -87,5 +88,5 @@
   </link>
   <link
-    name="body_upper_link">
+    name="$(arg robot)/body_upper_link">
     <inertial>
       <origin
@@ -127,5 +128,5 @@
   </link>
   <joint
-    name="body_bottom_j"
+    name="$(arg robot)/body_bottom_j"
     type="fixed">
     <origin
@@ -133,15 +134,15 @@
       rpy="1.5707963267949 0 0" />
     <parent
-      link="body_bott_link" />
-    <child
-      link="body_upper_link" />
+      link="$(arg robot)/body_bott_link" />
+    <child
+      link="$(arg robot)/body_upper_link" />
     <axis
       xyz="0 0 0" />
   </joint>
   <!-- FAKE FORWARD WHEEL -->
-  <link name="fake_fwd_wheel_link"/>
-  <joint name="fake_fwd_wheel_j" type="revolute">
-      <parent link="body_upper_link"/>
-      <child link="fake_fwd_wheel_link"/>
+  <link name="$(arg robot)/fake_fwd_wheel_link"/>
+  <joint name="$(arg robot)/fake_fwd_wheel_j" type="revolute">
+      <parent link="$(arg robot)/body_upper_link"/>
+      <child link="$(arg robot)/fake_fwd_wheel_link"/>
       <origin
           xyz="-0.1 -0.054 0"
@@ -157,5 +158,5 @@
   <!-- FORWARD LEFT WHEEL -->
   <link
-    name="fwd_left_wheel_holder_link">
+    name="$(arg robot)/fwd_left_wheel_holder_link">
     <inertial>
       <origin
@@ -197,5 +198,5 @@
   </link>
   <joint
-    name="fwd_left_wheel_holder_j"
+    name="$(arg robot)/fwd_left_wheel_holder_j"
     type="revolute">
     <origin
@@ -203,7 +204,7 @@
       rpy="0 0 0.035451" />
     <parent
-      link="body_upper_link" />
-    <child
-      link="fwd_left_wheel_holder_link" />
+      link="$(arg robot)/body_upper_link" />
+    <child
+      link="$(arg robot)/fwd_left_wheel_holder_link" />
     <axis
       xyz="0 1 0" />
@@ -218,5 +219,5 @@
   </joint>
   <link
-    name="fwd_left_wheel_link">
+    name="$(arg robot)/fwd_left_wheel_link">
     <inertial>
       <origin
@@ -259,5 +260,5 @@
   </link>
   <joint
-    name="fwd_left_wheel_j"
+    name="$(arg robot)/fwd_left_wheel_j"
     type="continuous">
     <origin
@@ -265,7 +266,7 @@
       rpy="1.5708 0 1.5353" />
     <parent
-      link="fwd_left_wheel_holder_link" />
-    <child
-      link="fwd_left_wheel_link" />
+      link="$(arg robot)/fwd_left_wheel_holder_link" />
+    <child
+      link="$(arg robot)/fwd_left_wheel_link" />
     <axis
       xyz="0 -1 0" />
@@ -274,10 +275,10 @@
       friction="0.01" />
   </joint>
-  <transmission name="tran_fwd_left_steer">
+  <transmission name="$(arg robot)/tran_fwd_left_steer">
     <type>transmission_interface/SimpleTransmission</type>
-    <joint name="fwd_left_wheel_holder_j">
+    <joint name="$(arg robot)/fwd_left_wheel_holder_j">
         <hardwareInterface>VelocityJointInterface</hardwareInterface>
     </joint>
-    <actuator name="fwd_left_steer">
+    <actuator name="$(arg robot)/fwd_left_steer">
         <hardwareInterface>VelocityJointInterface</hardwareInterface>
         <mechanicalReduction>1</mechanicalReduction>
@@ -296,5 +297,5 @@
   <!-- FORWARD RIGHT WHEEL -->
   <link
-    name="fwd_right_wheel_holder_link">
+    name="$(arg robot)/fwd_right_wheel_holder_link">
     <inertial>
       <origin
@@ -336,5 +337,5 @@
   </link>
   <joint
-    name="fwd_right_wheel_holder_j"
+    name="$(arg robot)/fwd_right_wheel_holder_j"
     type="revolute">
     <origin
@@ -342,7 +343,7 @@
       rpy="3.1416 0 3.1416" />
     <parent
-      link="body_upper_link" />
-    <child
-      link="fwd_right_wheel_holder_link" />
+      link="$(arg robot)/body_upper_link" />
+    <child
+      link="$(arg robot)/fwd_right_wheel_holder_link" />
     <axis
       xyz="0 1 0" />
@@ -357,5 +358,5 @@
   </joint>
   <link
-    name="fwd_right_wheel_link">
+    name="$(arg robot)/fwd_right_wheel_link">
     <inertial>
       <origin
@@ -398,5 +399,5 @@
   </link>
   <joint
-    name="fwd_right_wheel_j"
+    name="$(arg robot)/fwd_right_wheel_j"
     type="continuous">
     <origin
@@ -404,7 +405,7 @@
       rpy="1.5708 0 3.1416" />
     <parent
-      link="fwd_right_wheel_holder_link" />
-    <child
-      link="fwd_right_wheel_link" />
+      link="$(arg robot)/fwd_right_wheel_holder_link" />
+    <child
+      link="$(arg robot)/fwd_right_wheel_link" />
     <axis
       xyz="0 1 0" />
@@ -413,10 +414,10 @@
       friction="0.01" />
   </joint>
-  <transmission name="tran_fwd_right_steer">
+  <transmission name="$(arg robot)/tran_fwd_right_steer">
     <type>transmission_interface/SimpleTransmission</type>
-    <joint name="fwd_right_wheel_holder_j">
+    <joint name="$(arg robot)/fwd_right_wheel_holder_j">
         <hardwareInterface>VelocityJointInterface</hardwareInterface>
     </joint>
-    <actuator name="fwd_right_steer">
+    <actuator name="$(arg robot)/fwd_right_steer">
         <hardwareInterface>VelocityJointInterface</hardwareInterface>
         <mechanicalReduction>1</mechanicalReduction>
@@ -434,16 +435,16 @@
   </transmission>-->
   <!-- FAKE BACK LINK -->
-  <link name="fake_back_wheel_link"/>
-  <joint name="fake_back_wheel_j" type="continuous">
+  <link name="$(arg robot)/fake_back_wheel_link"/>
+  <joint name="$(arg robot)/fake_back_wheel_j" type="continuous">
          <origin
              xyz="0.1 -0.054 0.0"
              rpy="${pi/2} 0 ${pi}"/>
-         <parent link="body_upper_link"/>
-         <child link="fake_back_wheel_link"/>
+         <parent link="$(arg robot)/body_upper_link"/>
+         <child link="$(arg robot)/fake_back_wheel_link"/>
          <axis xyz="0 1 0"/>
      </joint>
   <!-- BACK LEFT WHEEL -->
   <link
-    name="back_left_wheel_holder_link">
+    name="$(arg robot)/back_left_wheel_holder_link">
     <inertial>
       <origin
@@ -485,5 +486,5 @@
   </link>
   <joint
-    name="back_left_wheel_holder_j"
+    name="$(arg robot)/back_left_wheel_holder_j"
     type="fixed">
     <origin
@@ -491,12 +492,12 @@
       rpy="0 0 0" />
     <parent
-      link="body_upper_link" />
-    <child
-      link="back_left_wheel_holder_link" />
+      link="$(arg robot)/body_upper_link" />
+    <child
+      link="$(arg robot)/back_left_wheel_holder_link" />
     <axis
       xyz="0 0 0" />
   </joint>
   <link
-    name="back_left_wheel_link">
+    name="$(arg robot)/back_left_wheel_link">
     <inertial>
       <origin
@@ -539,5 +540,5 @@
   </link>
   <joint
-    name="back_left_wheel_j"
+    name="$(arg robot)/back_left_wheel_j"
     type="continuous">
     <origin
@@ -545,7 +546,7 @@
       rpy="1.5708 0 0" />
     <parent
-      link="back_left_wheel_holder_link" />
-    <child
-      link="back_left_wheel_link" />
+      link="$(arg robot)/back_left_wheel_holder_link" />
+    <child
+      link="$(arg robot)/back_left_wheel_link" />
     <axis
       xyz="0 1 0" />
@@ -554,20 +555,20 @@
       friction="0.05" />
   </joint>
-  <transmission name="tran_back_left">
+  <transmission name="$(arg robot)/tran_back_left">
     <type>transmission_interface/SimpleTransmission</type>
-    <joint name="back_left_wheel_j">
+    <joint name="$(arg robot)/back_left_wheel_j">
         <hardwareInterface>VelocityJointInterface</hardwareInterface>
     </joint>
-    <actuator name="back_left">
+    <actuator name="$(arg robot)/back_left">
         <hardwareInterface>VelocityJointInterface</hardwareInterface>
         <mechanicalReduction>1</mechanicalReduction>
     </actuator>
   </transmission>
-  <transmission name="tran1">
+  <transmission name="$(arg robot)/tran1">
       <type>transmission_interface/SimpleTransmission</type>
-        <joint name="back_left_wheel_j">
+        <joint name="$(arg robot)/back_left_wheel_j">
           <hardwareInterface>EffortJointInterface</hardwareInterface>
         </joint>
-        <actuator name="motor1">
+        <actuator name="$(arg robot)/motor1">
           <hardwareInterface>EffortJointInterface</hardwareInterface>
           <mechanicalReduction>1</mechanicalReduction>
@@ -576,5 +577,5 @@
   <!-- BACK RIGHT WHEEL -->
   <link
-    name="back_right_wheel_holder_link">
+    name="$(arg robot)/back_right_wheel_holder_link">
     <inertial>
       <origin
@@ -616,5 +617,5 @@
   </link>
   <joint
-    name="back_right_wheel_holder_j"
+    name="$(arg robot)/back_right_wheel_holder_j"
     type="fixed">
     <origin
@@ -622,12 +623,12 @@
       rpy="3.1416 0 3.1416" />
     <parent
-      link="body_upper_link" />
-    <child
-      link="back_right_wheel_holder_link" />
+      link="$(arg robot)/body_upper_link" />
+    <child
+      link="$(arg robot)/back_right_wheel_holder_link" />
     <axis
       xyz="0 0 0" />
   </joint>
   <link
-    name="back_right_wheel_link">
+    name="$(arg robot)/back_right_wheel_link">
     <inertial>
       <origin
@@ -670,5 +671,5 @@
   </link>
   <joint
-    name="back_right_wheel_j"
+    name="$(arg robot)/back_right_wheel_j"
     type="continuous">
     <origin
@@ -676,7 +677,7 @@
       rpy="1.5708 0 1.5708" />
     <parent
-      link="back_right_wheel_holder_link" />
-    <child
-      link="back_right_wheel_link" />
+      link="$(arg robot)/back_right_wheel_holder_link" />
+    <child
+      link="$(arg robot)/back_right_wheel_link" />
     <axis
       xyz="0 -1 0" />
@@ -685,20 +686,20 @@
       friction="0.05" />
   </joint>
-  <transmission name="tran_back_right">
+  <transmission name="$(arg robot)/tran_back_right">
     <type>transmission_interface/SimpleTransmission</type>
-    <joint name="back_right_wheel_j">
+    <joint name="$(arg robot)/back_right_wheel_j">
         <hardwareInterface>VelocityJointInterface</hardwareInterface>
     </joint>
-    <actuator name="back_right">
+    <actuator name="$(arg robot)/back_right">
         <hardwareInterface>VelocityJointInterface</hardwareInterface>
         <mechanicalReduction>1</mechanicalReduction>
     </actuator>
   </transmission>
-  <transmission name="tran2">
+  <transmission name="$(arg robot)/tran2">
       <type>transmission_interface/SimpleTransmission</type>
-        <joint name="back_right_wheel_j">
+        <joint name="$(arg robot)/back_right_wheel_j">
           <hardwareInterface>EffortJointInterface</hardwareInterface>
         </joint>
-        <actuator name="motor2">
+        <actuator name="$(arg robot)/motor2">
           <hardwareInterface>EffortJointInterface</hardwareInterface>
           <mechanicalReduction>1</mechanicalReduction>

Commit message: robots don't see eachother with laser

File: mse6_description/urdf/mse6.xacro (robot description, xacro)
@@ -11,5 +11,14 @@
   <link name="$(arg robot)/base_link"/>
   <!-- SENSORS -->
-  <link name="$(arg robot)/laser_scanner_link"/>
+  <link name="$(arg robot)/laser_scanner_link">
+    <!--<collision>
+      <origin
+        xyz="0 0 0"
+        rpy="0 0 0" />
+      <geometry>
+          <box size="0.4 0.15 0.3" />
+      </geometry>
+    </collision>-->
+  </link>
   <joint name="$(arg robot)/laser_scanner_j"
          type="fixed">
@@ -84,4 +93,5 @@
         <mesh
           filename="package://mse6_description/meshes/body_bott_link.STL" />
+          <!--<box size="0.4 0.15 0.3" />-->
       </geometry>
     </collision>
